File: kicad/carte_raspi.sch (KiCad schematic (older format))
At the start: 24 parts, among them P1 CONN_2, P10 CONN_2, P11 CONN_2, P12 CONN_2, P13 CONN_2, P14 CONN_2, P15 CONN_2, P16 CONN_2, P17 CONN_2, P18 CONN_4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

Commit message: Some modifications on the connecting boar
Parts:
- removed P18: CONN_4, symbol CONN_4
- added P18: CONN_5, symbol CONN_5
Connections:
- net GND: now also P18.5
- net GPIO0: now also P18.1
- net GPIO1: now also P18.2
- net GPIO21: now also P18.4
- net GPIO5: now also P18.3
